Commit message: test

File: resources/robots/pointfoot/PF_TRON1A/urdf/robot.urdf (robot description, URDF)
Before this commit: robot point_foot, 12 links, 11 joints
Links:
- link abad_L_Link: geometry collision cylinder length=0.05 radius=0.05; visual mesh filename=meshes/abad_L_Link.STL
- link abad_R_Link: geometry collision cylinder length=0.05 radius=0.05; visual mesh filename=meshes/abad_R_Link.STL
- link base_Link: geometry collision box size=0.37 0.26 0.14; visual mesh filename=meshes/base_Link.STL
- link foot_L_Link: geometry collision sphere radius=0.03; visual mesh filename=meshes/foot_L_Link.STL
- link foot_R_Link: geometry collision sphere radius=0.03; visual mesh filename=meshes/foot_R_Link.STL
- link hip_L_Link: geometry collision cylinder length=0.15 radius=0.035; visual mesh filename=meshes/hip_L_Link.STL
- link hip_R_Link: geometry collision cylinder length=0.15 radius=0.035; visual mesh filename=meshes/hip_R_Link.STL
- link knee_L_Link: geometry collision cylinder length=0.26 radius=0.015; visual mesh filename=meshes/knee_L_Link.STL
- link knee_R_Link: geometry collision cylinder length=0.26 radius=0.015; visual mesh filename=meshes/knee_R_Link.STL
